Commit message: correct package name

File: ws/src/camera_simulations/robot/aruco_seven_dof_arm_with_rgbd.xacro (robot description, xacro)
@@ -381,5 +381,5 @@
         <pose>0 0 0 0 0 0</pose>
         <geometry>
-          <mesh filename="$(find gazebo_sensors_tutorial)/models/aruco_cube/meshes/aruco_cube_5cm.dae">
+          <mesh filename="$(find camera_simulations)/models/aruco_cube/meshes/aruco_cube_5cm.dae">
           </mesh>
         </geometry>
@@ -400,5 +400,5 @@
       <origin xyz="0.08 0 0" rpy="0 0 0"/>
     </joint>
-  <xacro:include filename="$(find gazebo_sensors_tutorial)/robot/sensors/xtion_pro_live.urdf.xacro"/>
+  <xacro:include filename="$(find camera_simulations)/robot/sensors/xtion_pro_live.urdf.xacro"/>
 <!-- ///////////////////////////////////////////////////////////////////////////////////////////////////////////////////// -->
   <!-- Transmissions for ROS Control -->

File: ws/src/camera_simulations/robot/camera_left.urdf.xacro (robot description, xacro)
@@ -1,6 +1,6 @@
 <?xml version="1.0"?>
 <robot xmlns:xacro="http://ros.org/wiki/xacro" name="camera_left">
-	<xacro:include filename="$(find gazebo_sensors_tutorial)/robot/sensors/_d415.urdf.xacro"/>
-	<xacro:include filename="$(find gazebo_sensors_tutorial)/robot/sensors/cam_holder.urdf.xacro"/>
+	<xacro:include filename="$(find camera_simulations)/robot/sensors/_d415.urdf.xacro"/>
+	<xacro:include filename="$(find camera_simulations)/robot/sensors/cam_holder.urdf.xacro"/>
 	<link name="chess_frame" />
         <!-- sets camera frame w.r.t. to chess frame-->

File: ws/src/camera_simulations/robot/camera_right.urdf.xacro (robot description, xacro)
@@ -1,6 +1,6 @@
 <?xml version="1.0"?>
 <robot xmlns:xacro="http://ros.org/wiki/xacro" name="camera_right">
-	<xacro:include filename="$(find gazebo_sensors_tutorial)/robot/sensors/_d415.urdf.xacro"/>
-	<xacro:include filename="$(find gazebo_sensors_tutorial)/robot/sensors/cam_holder.urdf.xacro"/>
+	<xacro:include filename="$(find camera_simulations)/robot/sensors/_d415.urdf.xacro"/>
+	<xacro:include filename="$(find camera_simulations)/robot/sensors/cam_holder.urdf.xacro"/>
 	<link name="chess_frame" />
         <!-- sets camera frame w.r.t. to chess frame-->
